File: X16-ESC-Controller.sch (EAGLE design)
At the start: 6 parts

Commit message: STM & Connectors
Parts:
- added C3: 4.7uF, SparkFun-Capacitors:4.7PF-0603-50V-5%
- added C4: 0.1uF, SparkFun-Capacitors:4.7PF-0603-50V-5%
- added D1: Green, SparkFun-LED:LED-GREEN-0603-WE
- added J1, J2: (no value), SparkFun-Connectors:CONN_06NO_SILK_NO_POP
- added R2: 1k, SparkFun-Resistors:2.55KOHM-0603-1/10W-1%
- added U$3: (no value), X16-ESC-Controller:SWITCH_DISCRETECOMPONENTS
- added U$4: CONN_BAKCPLANE, X16-ESC-Controller:CONN_BAKCPLANE
- C2: value 4.7pF -> 4.7uF
Connections:
- new net ESC_ID: U$1.12
- new net N$10: J1.4
- new net N$11: J1.3
- new net N$12: J1.2
- new net N$13: J1.1
- new net N$17: J2.2
- new net N$3: R2.1, U$2.PB6
- new net N$7: D1.A, R2.2
- new net N$9: J1.5
- new net NRST: U$1.6
- new net SPI: U$1.5, U$1.7
- net ADC_IN4: now also J2.1
- net GND: now also C3.2, C4.2, U$1.10, U$3.P$1
- net N$2: now also C3.1, U$3.P$2
- net SWCLK: now also U$1.11
- net SWDIO: now also U$1.9
- net TIM16_CH1: now also J2.3
- net TIM3_CH2: now also J2.4
- net TIM3_CH3: now also J2.5
- net TIM3_CH4: now also J1.6, J2.6
- net VCC: now also C4.1, R1.1, U$1.1, U$1.2, U$1.3, U$1.4, U$2.VDDA
Other:
- moved on the sheet: U$1

Commit message: schematic
Parts:
- added C5: 22uF, SparkFun-Capacitors:4.7PF-0603-50V-5%
- added C7: 10uF, SparkFun-Capacitors:4.7PF-0603-50V-5%
- added D2: Green, SparkFun-LED:LED-GREEN-0603-WE
- added IC1: OP-AMP, SparkFun-IC-Amplifiers:OPAMP-DUALU
- added J3: 455-1750-1-ND, SparkFun-Connectors:CONN_03
- added JP1: JUMPER-SMT_2_NC_TRACE_NO-SILK, SparkFun-Jumpers:JUMPER-SMT_2_NC_TRACE_NO-SILK
- added R3: 3.3k, SparkFun-Resistors:2.55KOHM-0603-1/10W-1%
- added R4: 1k, SparkFun-Resistors:2.55KOHM-0603-1/10W-1%
- added R6: 150, SparkFun-Resistors:2.55KOHM-0603-1/10W-1%
- added U1: AZ1117IH-3.3TRG1, X16-ESC-Controller:AZ1117IH-3.3TRG1
Connections:
- net ESC_ID renamed PWM4
- net NRST renamed PWM1
- removed net N$10: J1.4
- removed net N$11: J1.3
- removed net N$13: J1.1
- removed net N$4: U$2.PA12
- removed net N$6: U$2.PA11
- removed net N$9: J1.5
- removed net SPI: U$1.5, U$1.7
- new net CS: U$1.11
- new net MISO: U$1.5, U$2.PA11
- new net MOSI: U$1.7, U$2.PA12
- new net N$14: IC1G1.+IN, JP1.1
- new net N$15: IC1G1.-IN, R3.2, R4.1
- new net N$16: D2.A, R6.2
- new net N$8: IC1G1.OUT, JP1.2
- new net PWM2: U$1.8
- new net PWM3: U$1.10
- new net SCLK: U$1.9
- new net TIM14_CH1: J3.1
- net ADC_IN1: now also J1.1
- net GND: now also C5.1, C7.2, IC1G3.P$V-, R3.1, R6.1, U$1.2, U$1.4, U1.ADJ/GND; no longer U$1.10
- net SWCLK: now also U$4.3; no longer U$1.11
- net SWDIO: now also U$4.1; no longer U$1.9
- net TIM16_CH1: now also J3.2
- net TIM17_CH1: now also J3.3
- net TIM2_CH1: now also J1.3
- net TIM2_CH2: now also J1.4
- net TIM2_CH3: now also J1.5
- net TIM2_CH4: now also J1.6
- net TIM3_CH4: no longer J1.6
- net VCC: now also C5.2, C7.1, IC1G3.P$V+, R4.2, U1.INPUT, U1.OUTPUT; no longer U$1.2, U$1.4
Other:
- moved on the sheet: C1, C2, C3, C4, C6, D1, J1, J2, R1, R2, U$1, U$2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

Commit message: final?
Parts:
- removed IC1: OP-AMP, SparkFun-IC-Amplifiers:OPAMP-DUALU
- removed J3: 455-1750-1-ND, SparkFun-Connectors:CONN_03
- removed JP1: JUMPER-SMT_2_NC_TRACE_NO-SILK, SparkFun-Jumpers:JUMPER-SMT_2_NC_TRACE_NO-SILK
- removed R3: 3.3k, SparkFun-Resistors:2.55KOHM-0603-1/10W-1%
- removed R4: 1k, SparkFun-Resistors:2.55KOHM-0603-1/10W-1%
- removed U$1, U$4: CONN_BAKCPLANE, X16-ESC-Controller:CONN_BAKCPLANE
- added J4: (no value), SparkFun-Connectors:CONN_05LOCK_LONGPADS
- added J5: (no value), SparkFun-Connectors:CONN_02
- added J6: TMMH-110-05-F-D, TMMH-110-05-F-D:TMMH-110-05-F-D
- added TP1, TP10, TP11, TP12, TP13, TP2, TP3, TP4, TP6, TP7, TP8, TP9: TEST-POINT3, SparkFun-Connectors:TEST-POINT3
- C5: value 22uF -> 4.7uF
- C7: value 10uF -> 4.7uF
Connections:
- removed net ADC_IN0: U$2.PA0
- removed net ADC_IN1: J1.1, U$2.PA1
- removed net ADC_IN4: J2.1, U$2.PA4
- removed net N$12: J1.2
- removed net N$14: IC1G1.+IN, JP1.1
- removed net N$15: IC1G1.-IN, R3.2, R4.1
- removed net N$17: J2.2
- removed net N$8: IC1G1.OUT, JP1.2
- removed net PWM1: U$1.6
- removed net PWM2: U$1.8
- removed net PWM3: U$1.10
- removed net PWM4: U$1.12
- removed net TIM14_CH1: J3.1
- removed net TIM16_CH1: J2.3, J3.2, U$2.PA15
- removed net TIM17_CH1: J3.3, U$2.PA7
- new net NRST: J4.1
- new net PWMA0: J6.13
- new net PWMA1: J6.15
- new net PWMA2: J6.17
- new net PWMA3: J6.19
- new net PWMB0: J6.06
- new net PWMB1: J6.08
- new net PWMB2: J6.10
- new net PWMB3: J6.12
- new net PWMC0: J6.14
- new net PWMC1: J6.16
- new net PWMC2: J6.18
- new net PWMC3: J6.20
- new net SPI1_MISO: U$2.PA6
- new net SPI1_MOSI: U$2.PA7
- new net SPI1_NSS: U$2.PA4
- new net SPI1_SCK: U$2.PA5
- new net SYS_SWCLK: U$2.PA14
- new net SYS_SWDIO: U$2.PA13
- new net TIM1_CH4: J2.2, TP10.1, U$2.PA11
- new net TIM3_CH1: J2.3, TP9.1, U$2.PB4
- net CS: now also J6.11; no longer U$1.11
- net GND: now also J4.3, J5.1, J6.02, J6.04; no longer IC1G3.P$V-, R3.1, U$1.2, U$1.4
- net MISO: now also J6.05; no longer U$1.5, U$2.PA11
- net MOSI: now also J6.07; no longer U$1.7, U$2.PA12
- net SCLK: now also J6.09; no longer U$1.9
- net SWCLK: now also J4.4; no longer U$2.PA14, U$4.3
- net SWDIO: now also J4.2; no longer U$2.PA13, U$4.1
- net TIM1_CH1: now also J1.1, TP11.1
- net TIM1_CH2: now also J1.2, TP12.1
- net TIM1_CH3: now also J2.1, TP13.1
- net TIM2_CH1: now also TP1.1, U$2.PA0; no longer U$2.PB3
- net TIM2_CH2: now also TP4.1, U$2.PA1; no longer U$2.PB4
- net TIM2_CH3: now also TP3.1
- net TIM2_CH4: now also TP2.1
- net TIM3_CH2: now also TP8.1
- net TIM3_CH3: now also TP7.1
- net TIM3_CH4: now also TP6.1
- net VCC: now also D2.C, J4.5, J5.2, J6.01, J6.03; no longer IC1G3.P$V+, R4.2, U$1.1, U$1.3
Other:
- note added: "Backplane Connector"
- note added: "Indicating LED"
- note added: "Program Header Pins"
- note added: "Regulator"
- note added: "Test Points"
- note added: "Timer Channels"
- moved on the sheet: C1, C2, C3, C4, C5, C6, C7, D1, D2, J1, J2, R1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

Commit message: 11/4/2023
Connections:
- removed net N$5: U$2.PB7
- removed net PWMA0: J6.13
- removed net PWMA1: J6.15
- removed net PWMA2: J6.17
- removed net PWMA3: J6.19
- removed net PWMB0: J6.06
- removed net PWMB1: J6.08
- removed net PWMB2: J6.10
- removed net PWMB3: J6.12
- removed net PWMC0: J6.14
- removed net PWMC1: J6.16
- removed net PWMC2: J6.18
- removed net PWMC3: J6.20
- removed net SYS_SWCLK: U$2.PA14
- removed net SYS_SWDIO: U$2.PA13
- new net 3V3: C1.1, C2.1, C4.1, C6.1, C7.1, D2.C, J5.2, R1.1, U$2.VDD, U$2.VDDA, U$2.VDDIO2, U1.OUTPUT
- new net 5.2V: C5.2, J6.01, J6.03, U1.INPUT
- net SWCLK: now also U$2.PA14
- net SWDIO: now also U$2.PA13
- net TIM1_CH1: now also J6.13
- net TIM1_CH2: now also J6.15
- net TIM1_CH3: now also J6.17
- net TIM1_CH4: now also J6.19
- net TIM2_CH1: now also J6.06
- net TIM2_CH2: now also J6.08
- net TIM2_CH3: now also J6.10
- net TIM2_CH4: now also J6.12
- net TIM3_CH1: now also J6.14
- net TIM3_CH2: now also J6.16
- net TIM3_CH3: now also J6.18
- net TIM3_CH4: now also J6.20
- net VCC: no longer C1.1, C2.1, C4.1, C5.2, C6.1, C7.1, D2.C, J5.2, J6.01, J6.03, R1.1, U$2.VDD, U$2.VDDA, U$2.VDDIO2, U1.INPUT, U1.OUTPUT
Other:
- note added: "STM"
- moved on the sheet: C1, C2, C3, C4, C5, C6, C7, D1, D2, J1, J2, J4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

Commit message: 11/04/23
Parts:
- removed TP2: TEST-POINT3, SparkFun-Connectors:TEST-POINT3
- added FGFD: TEST-POINT3, SparkFun-Connectors:TEST-POINT3
Connections:
- removed net N$1: U$2.PB8-BOOT0, U$2.VSS1
- removed net N$2: C3.1, R1.2, U$2.NRST, U$3.P$2
- removed net SPI1_MISO: U$2.PA6
- removed net SPI1_MOSI: U$2.PA7
- removed net SPI1_NSS: U$2.PA4
- removed net SPI1_SCK: U$2.PA5
- removed net VCC: J4.5
- net 3V3: now also J4.5
- net CS: now also U$2.PA4
- net GND: now also D1.C, U$2.PB8-BOOT0, U$2.VSS1
- net MISO: now also U$2.PA6
- net MOSI: now also U$2.PA7
- net NRST: now also C3.1, R1.2, U$2.NRST, U$3.P$2
- net SCLK: now also U$2.PA5
- net TIM2_CH4: now also FGFD.1; no longer TP2.1
Other:
- moved on the sheet: C1, C2

Commit message: 11/08/23
Parts:
- removed FGFD, TP10, TP11, TP12, TP13, TP4, TP6, TP7, TP8, TP9: TEST-POINT3, SparkFun-Connectors:TEST-POINT3
- added TP2: (no value), SparkFun-Connectors:CONN_01
- TP1, TP3: value TEST-POINT3 -> (none); device SparkFun-Connectors:TEST-POINT3 -> SparkFun-Connectors:CONN_01
Connections:
- net 3V3: now also TP1.1
- net 5.2V: now also TP2.1
- net GND: now also TP3.1
- net TIM1_CH1: no longer TP11.1
- net TIM1_CH2: no longer TP12.1
- net TIM1_CH3: no longer TP13.1
- net TIM1_CH4: no longer TP10.1
- net TIM2_CH1: no longer TP1.1
- net TIM2_CH2: no longer TP4.1
- net TIM2_CH3: no longer TP3.1
- net TIM2_CH4: no longer FGFD.1
- net TIM3_CH1: no longer TP9.1
- net TIM3_CH2: no longer TP8.1
- net TIM3_CH3: no longer TP7.1
- net TIM3_CH4: no longer TP6.1

Commit message: 11/16/23
Parts:
- J4: device SparkFun-Connectors:CONN_05LOCK_LONGPADS -> SparkFun-Connectors:CONN_05LOCK
Changed lines of the file:
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@@
 <part name="C7" library="SparkFun-Capacitors" library_urn="urn:adsk.eagle:library:510" deviceset="4.7PF" device="-0603-50V-5%" package3d_urn="urn:adsk.eagle:package:41385090/1" value="4.7uF"/>
 <part name="GND15" library="SparkFun-PowerSymbols" library_urn="urn:adsk.eagle:library:530" deviceset="GND" device=""/>
-<part name="J4" library="SparkFun-Connectors" library_urn="urn:adsk.eagle:library:513" deviceset="CONN_05" device="LOCK_LONGPADS" package3d_urn="urn:adsk.eagle:package:38107/2"/>
+<part name="J4" library="SparkFun-Connectors" library_urn="urn:adsk.eagle:library:513" deviceset="CONN_05" device="LOCK" package3d_urn="urn:adsk.eagle:package:38105/2"/>
 <part name="J5" library="SparkFun-Connectors" library_urn="urn:adsk.eagle:library:513" deviceset="CONN_02" device="" package3d_urn="urn:adsk.eagle:package:38039/2"/>
 <part name="GND16" library="SparkFun-PowerSymbols" library_urn="urn:adsk.eagle:library:530" deviceset="GND" device=""/>
