File: X16-ESC-Controller.brd (EAGLE design)
At the start: 160 x 100 mm, 6 parts

Commit message: STM & Connectors
Parts:
- added C3: 4.7uF, SparkFun-Capacitors:0603
- added C4: 0.1uF, SparkFun-Capacitors:0603
- added U$3: (no value), X16-ESC-Controller:DISCRETECOMPONENTS_SW_2512
- C2: value 4.7pF -> 4.7uF
Connections:
- net GND: now also C3.2, C4.2, U$3.1
- net N$2: now also C3.1, U$3.2
- net VCC: now also C4.1, R1.1, U$2.VDDA
Changed lines of the file:
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@@
 <attribute name="VALUE" x="-15.24" y="-7.112" size="0.6096" layer="27" font="vector" ratio="20" align="top-center"/>
 </element>
-<element name="C2" library="SparkFun-Capacitors" library_urn="urn:adsk.eagle:library:510" package="0603" package3d_urn="urn:adsk.eagle:package:41385090/1" value="4.7pF" x="-15.24" y="-10.16" smashed="yes">
+<element name="C2" library="SparkFun-Capacitors" library_urn="urn:adsk.eagle:library:510" package="0603" package3d_urn="urn:adsk.eagle:package:41385090/1" value="4.7uF" x="-15.24" y="-10.16" smashed="yes">
 <attribute name="NAME" x="-15.24" y="-9.398" size="0.6096" layer="25" font="vector" ratio="20" align="bottom-center"/>
 <attribute name="PROD_ID" value="CAP-07880" x="-15.24" y="-10.16" size="1.778" layer="27" display="off"/>
@@
 <attribute name="VALUE" x="-15.24" y="-14.732" size="0.6096" layer="27" font="vector" ratio="20" align="top-center"/>
 </element>
+<element name="C3" library="SparkFun-Capacitors" library_urn="urn:adsk.eagle:library:510" package="0603" package3d_urn="urn:adsk.eagle:package:41385090/1" value="4.7uF" x="-15.24" y="-17.78" smashed="yes">
+<attribute name="NAME" x="-15.24" y="-17.018" size="0.6096" layer="25" font="vector" ratio="20" align="bottom-center"/>
+<attribute name="PROD_ID" value="CAP-07880" x="-15.24" y="-17.78" size="1.778" layer="27" display="off"/>
+<attribute name="VALUE" x="-15.24" y="-18.542" size="0.6096" layer="27" font="vector" ratio="20" align="top-center"/>
+</element>
+<element name="U$3" library="X16-ESC-Controller" package="DISCRETECOMPONENTS_SW_2512" package3d_urn="urn:adsk.eagle:package:24384574/2" value="" x="-12.7" y="-24.13" smashed="yes">
+<attribute name="NAME" x="-12.7" y="-22.225" size="1.27" layer="25" align="bottom-center"/>
+<attribute name="VALUE" x="-12.7" y="-26.035" size="1.27" layer="27" align="top-center"/>
+</element>
+<element name="C4" library="SparkFun-Capacitors" library_urn="urn:adsk.eagle:library:510" package="0603" package3d_urn="urn:adsk.eagle:package:41385090/1" value="0.1uF" x="-15.24" y="-27.94" smashed="yes">
+<attribute name="NAME" x="-15.24" y="-27.178" size="0.6096" layer="25" font="vector" ratio="20" align="bottom-center"/>
+<attribute name="PROD_ID" value="CAP-07880" x="-15.24" y="-27.94" size="1.778" layer="27" display="off"/>
+<attribute name="VALUE" x="-15.24" y="-28.702" size="0.6096" layer="27" font="vector" ratio="20" align="top-center"/>
+</element>
 </elements>
 <signals>
@@
 <contactref element="C1" pad="2"/>
 <contactref element="C2" pad="2"/>
+<contactref element="U$3" pad="1"/>
+<contactref element="C3" pad="2"/>
+<contactref element="C4" pad="2"/>
+<wire x1="-15.7" y1="-24.13" x2="-14.39" y2="-27.94" width="0" layer="19" extent="1-1"/>
+<wire x1="-14.39" y1="-17.78" x2="-15.7" y2="-24.13" width="0" layer="19" extent="1-1"/>
+<wire x1="-14.39" y1="-10.16" x2="-14.39" y2="-17.78" width="0" layer="19" extent="1-1"/>
 <wire x1="-14.39" y1="-6.35" x2="-14.39" y2="-10.16" width="0" layer="19" extent="1-1"/>
 <wire x1="-14.39" y1="-2.54" x2="-14.39" y2="-6.35" width="0" layer="19" extent="1-1"/>
@@
 <contactref element="C1" pad="1"/>
 <contactref element="C2" pad="1"/>
+<contactref element="R1" pad="1"/>
+<contactref element="C4" pad="1"/>
+<contactref element="U$2" pad="VDDA"/>
+<wire x1="-16.09" y1="-13.97" x2="-16.09" y2="-27.94" width="0" layer="19" extent="1-1"/>
+<wire x1="-16.09" y1="-10.16" x2="-16.09" y2="-13.97" width="0" layer="19" extent="1-1"/>
 <wire x1="-16.09" y1="-6.35" x2="-16.09" y2="-10.16" width="0" layer="19" extent="1-1"/>
 <wire x1="-16.09" y1="-2.54" x2="-16.09" y2="-6.35" width="0" layer="19" extent="1-1"/>
-<wire x1="-8.01" y1="2.54" x2="-16.09" y2="-2.54" width="0" layer="19" extent="1-1"/>
-<wire x1="-16.51" y1="8.14" x2="-8.01" y2="2.54" width="0" layer="19" extent="1-1"/>
+<wire x1="-16.51" y1="4.94" x2="-16.09" y2="-2.54" width="0" layer="19" extent="1-1"/>
+<wire x1="-16.51" y1="8.14" x2="-16.51" y2="4.94" width="0" layer="19" extent="1-1"/>
+<wire x1="-8.01" y1="2.54" x2="-16.51" y2="4.94" width="0" layer="19" extent="1-1"/>
 </signal>
 <signal name="N$2">
 <contactref element="U$2" pad="NRST"/>
 <contactref element="R1" pad="2"/>
+<contactref element="C3" pad="1"/>
+<contactref element="U$3" pad="2"/>
+<wire x1="-14.39" y1="-13.97" x2="-16.09" y2="-17.78" width="0" layer="19" extent="1-1"/>
+<wire x1="-9.7" y1="-24.13" x2="-16.09" y2="-17.78" width="0" layer="19" extent="1-1"/>
 <wire x1="-16.51" y1="5.74" x2="-14.39" y2="-13.97" width="0" layer="19" extent="1-1"/>
 </signal>

Commit message: testing
Parts:
- removed U$1: CONN_BAKCPLANE, X16-ESC-Controller:BACKPLANE_CONNECTORS_BKP
- added C5, C7: 4.7uF, SparkFun-Capacitors:0603
- added D1, D2: Green, SparkFun-LED:LED-0603
- added J1, J2: (no value), SparkFun-Connectors:1X06_NO_SILK
- added J4: (no value), SparkFun-Connectors:1X05_LOCK_LONGPADS
- added J5: (no value), SparkFun-Connectors:1X02
- added J6: TMMH-110-05-F-D, TMMH-110-05-F-D:SAMTEC_TMMH-110-05-F-D
- added R2: 1k, SparkFun-Resistors:0603
- added R6: 150, SparkFun-Resistors:0603
- added TP1, TP10, TP11, TP12, TP13, TP2, TP3, TP4, TP6, TP7, TP8, TP9: TEST-POINT3, SparkFun-Connectors:PAD.03X.03
- added U1: AZ1117IH-3.3TRG1, X16-ESC-Controller:SOT223_AZ1117I_6P5X3P5_DIO
- moved C4 75.0 mm to (-19.1, 47.0)
- moved C3 64.8 mm to (-15.2, 47.0)
- moved C2 64.1 mm to (-50.8, 43.2)
- moved R1 63.9 mm to (-34.3, 47.0)
- moved U$3 61.2 mm to (-17.8, 36.8)
- moved C1 58.8 mm to (-47.0, 43.2)
- moved C6 50.8 mm to (-26.7, 47.0)
- moved U$2 29.6 mm to (5.08, 22.9)
Connections:
- net ADC_IN4 renamed SPI1_NSS
- net TIM17_CH1 renamed SPI1_MOSI
- removed net ADC_IN0: U$2.PA0
- removed net ADC_IN1: U$2.PA1
- removed net N$4: U$2.PA12
- removed net N$6: U$2.PA11
- removed net TIM16_CH1: U$2.PA15
- new net CS: J6.11
- new net MISO: J6.05
- new net MOSI: J6.07
- new net N$16: D2.A, R6.2
- new net N$3: R2.1, U$2.PB6
- new net N$7: D1.A, R2.2
- new net NRST: J4.1
- new net PWMA0: J6.13
- new net PWMA1: J6.15
- new net PWMA2: J6.17
- new net PWMA3: J6.19
- new net PWMB0: J6.06
- new net PWMB1: J6.08
- new net PWMB2: J6.10
- new net PWMB3: J6.12
- new net PWMC0: J6.14
- new net PWMC1: J6.16
- new net PWMC2: J6.18
- new net PWMC3: J6.20
- new net SCLK: J6.09
- new net SPI1_MISO: U$2.PA6
- new net SPI1_SCK: U$2.PA5
- new net SYS_SWCLK: U$2.PA14
- new net SYS_SWDIO: U$2.PA13
- new net TIM1_CH4: J2.2, TP10.1, U$2.PA11
- new net TIM3_CH1: J2.3, TP9.1, U$2.PB4
- net GND: now also C5.1, C7.2, J4.3, J5.1, J6.02, J6.04, R6.1, U1.1
- net SWCLK: now also J4.4; no longer U$2.PA14
- net SWDIO: now also J4.2; no longer U$2.PA13
- net TIM1_CH1: now also J1.1, TP11.1
- net TIM1_CH2: now also J1.2, TP12.1
- net TIM1_CH3: now also J2.1, TP13.1
- net TIM2_CH1: now also J1.3, TP1.1, U$2.PA0; no longer U$2.PB3
- net TIM2_CH2: now also J1.4, TP4.1, U$2.PA1; no longer U$2.PB4
- net TIM2_CH3: now also J1.5, TP3.1
- net TIM2_CH4: now also J1.6, TP2.1
- net TIM3_CH2: now also J2.4, TP8.1
- net TIM3_CH3: now also J2.5, TP7.1
- net TIM3_CH4: now also J2.6, TP6.1
- net VCC: now also C5.2, C7.1, D2.C, J4.5, J5.2, J6.01, J6.03, U1.2, U1.3
Other:
- board size 160 x 100 mm -> 51.6 x 34.2 mm

Commit message: 11/4/2023
Connections:
- removed net N$5: U$2.PB7
- removed net PWMA0: J6.13
- removed net PWMA1: J6.15
- removed net PWMA2: J6.17
- removed net PWMA3: J6.19
- removed net PWMB0: J6.06
- removed net PWMB1: J6.08
- removed net PWMB2: J6.10
- removed net PWMB3: J6.12
- removed net PWMC0: J6.14
- removed net PWMC1: J6.16
- removed net PWMC2: J6.18
- removed net PWMC3: J6.20
- removed net SYS_SWCLK: U$2.PA14
- removed net SYS_SWDIO: U$2.PA13
- new net 3V3: C1.1, C2.1, C4.1, C6.1, C7.1, D2.C, J5.2, R1.1, U$2.VDD, U$2.VDDA, U$2.VDDIO2, U1.2
- new net 5.2V: C5.2, J6.01, J6.03, U1.3
- net SWCLK: now also U$2.PA14
- net SWDIO: now also U$2.PA13
- net TIM1_CH1: now also J6.13
- net TIM1_CH2: now also J6.15
- net TIM1_CH3: now also J6.17
- net TIM1_CH4: now also J6.19
- net TIM2_CH1: now also J6.06
- net TIM2_CH2: now also J6.08
- net TIM2_CH3: now also J6.10
- net TIM2_CH4: now also J6.12
- net TIM3_CH1: now also J6.14
- net TIM3_CH2: now also J6.16
- net TIM3_CH3: now also J6.18
- net TIM3_CH4: now also J6.20
- net VCC: no longer C1.1, C2.1, C4.1, C5.2, C6.1, C7.1, D2.C, J5.2, J6.01, J6.03, R1.1, U$2.VDD, U$2.VDDA, U$2.VDDIO2, U1.2, U1.3

Commit message: 11/04/23
Parts:
- moved J2 85.8 mm to (33.0, 2.54)
- moved J1 82.4 mm to (48.3, 7.62), turned to 90 degrees
- moved J4 73.9 mm to (33.0, 6.35)
- moved U$3 66.6 mm to (48.3, 27.9), turned to 90 degrees
- moved J5 50.6 mm to (5.08, 15.2), turned to 180 degrees
- renumbered TP2 to FGFD
Connections:
- removed net N$1: U$2.PB8-BOOT0, U$2.VSS1
- removed net N$2: C3.1, R1.2, U$2.NRST, U$3.2
- removed net SPI1_MISO: U$2.PA6
- removed net SPI1_MOSI: U$2.PA7
- removed net SPI1_NSS: U$2.PA4
- removed net SPI1_SCK: U$2.PA5
- removed net VCC: J4.5
- net 3V3: now also J4.5
- net CS: now also U$2.PA4
- net GND: now also D1.C, U$2.PB8-BOOT0, U$2.VSS1
- net MISO: now also U$2.PA6
- net MOSI: now also U$2.PA7
- net NRST: now also C3.1, R1.2, U$2.NRST, U$3.2
- net SCLK: now also U$2.PA5

Commit message: 11/08/23
Parts:
- removed FGFD, TP10, TP11, TP12, TP13, TP4, TP6, TP7, TP8, TP9: TEST-POINT3, SparkFun-Connectors:PAD.03X.03
- added TP2: (no value), SparkFun-Connectors:1X01
- TP1, TP3: value TEST-POINT3 -> (none); device SparkFun-Connectors:PAD.03X.03 -> SparkFun-Connectors:1X01
- moved C2 67.6 mm to (10.2, 14.0)
- moved C3 66.5 mm to (44.5, 17.8)
- moved C6 66.5 mm to (33.0, 17.8)
- moved C4 66.5 mm to (40.6, 17.8)
- moved C5 66.5 mm to (36.8, 17.8)
- moved C7 66.5 mm to (29.2, 17.8)
- moved D1 66.5 mm to (14.0, 17.8)
- moved D2 66.5 mm to (10.2, 17.8)
- moved R1 66.5 mm to (25.4, 17.8)
- moved R2 66.5 mm to (21.6, 17.8)
- moved R6 66.5 mm to (17.8, 17.8)
- moved TP1 65.7 mm to (-2.54, 3.81)
- moved C1 64.8 mm to (16.5, 30.5)
- moved TP3 47.1 mm to (-12.7, 3.81)
- moved U1 6.35 mm to (29.2, 29.2)
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Connections:
- net 3V3: now also TP1.1
- net 5.2V: now also TP2.1
- net GND: now also TP3.1
- net TIM1_CH1: no longer TP11.1
- net TIM1_CH2: no longer TP12.1
- net TIM1_CH3: no longer TP13.1
- net TIM1_CH4: no longer TP10.1
- net TIM2_CH1: no longer TP1.1
- net TIM2_CH2: no longer TP4.1
- net TIM2_CH3: no longer TP3.1
- net TIM2_CH4: no longer FGFD.1
- net TIM3_CH1: no longer TP9.1
- net TIM3_CH2: no longer TP8.1
- net TIM3_CH3: no longer TP7.1
- net TIM3_CH4: no longer TP6.1

Commit message: 11/16/23
Parts:
- J4: device SparkFun-Connectors:1X05_LOCK_LONGPADS -> SparkFun-Connectors:1X05_LOCK
- moved J5 47.1 mm to (48.9, 32.4), turned to 270 degrees
- moved TP3 31.1 mm to (2.16, 31.1)
- moved U$2 28.5 mm to (29.7, 15.5)
- moved J1 28.2 mm to (34.8, 32.4), turned to 180 degrees
- moved C5 27.8 mm to (9.14, 14.9), turned to 90 degrees
- moved D1 23.4 mm to (35.2, 27.6), turned to 180 degrees
- moved C2 23.3 mm to (33.3, 16.8), flipped to the bottom, turned to 90 degrees
- moved R6 21.0 mm to (2.03, 3.94), turned to 90 degrees
- moved C7 20.4 mm to (8.89, 18.9), turned to 90 degrees
- moved R1 19.7 mm to (44.3, 12.2), turned to 270 degrees
- moved J4 18.9 mm to (49.0, 16.4), turned to 90 degrees
- moved TP2 18.7 mm to (11.0, 2.67)
- moved U$3 18.7 mm to (48.9, 9.27)
- moved C1 18.0 mm to (31.2, 20.2), flipped to the bottom, turned to 270 degrees
- moved U1 17.9 mm to (15.2, 18.0), turned to 270 degrees
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Routing:
- net 3V3: track 0.00 -> 102.1 mm, vias 0 -> 5
- net TIM3_CH1: track 0.00 -> 49.5 mm
- net TIM1_CH1: track 0.00 -> 48.4 mm, vias 0 -> 2
- net TIM3_CH2: track 0.00 -> 46.4 mm
- net TIM1_CH2: track 0.00 -> 45.9 mm, vias 0 -> 1
- net NRST: track 0.00 -> 45.2 mm
- net TIM2_CH4: track 0.00 -> 43.7 mm, vias 0 -> 1
- net TIM2_CH1: track 0.00 -> 38.1 mm, vias 0 -> 1
- net TIM2_CH3: track 0.00 -> 37.8 mm, vias 0 -> 1
- net TIM2_CH2: track 0.00 -> 37.5 mm, vias 0 -> 1
- net GND: track 0.00 -> 32.8 mm, vias 0 -> 1
- net MISO: track 0.00 -> 32.7 mm, vias 0 -> 2
- net TIM3_CH3: track 0.00 -> 31.1 mm, vias 0 -> 1
- net TIM3_CH4: track 0.00 -> 29.6 mm
- net TIM1_CH4: track 0.00 -> 26.9 mm, vias 0 -> 1
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- added copper zone on layer 1, net GND
- added copper zone on layer 16, net GND

Commit message: 11/17/23
Parts:
- TP1, TP2, TP3: value (none) -> TESTPOINT_5.04MM; device SparkFun-Connectors:1X01 -> X16-ExtraComponents:TESTPOINT_5.04MM
- moved TP1 5.40 mm to (4.06, 22.9)
- moved TP2 3.37 mm to (7.87, 3.81)
- moved TP3 2.16 mm to (4.06, 30.1)
Connections:
- net 3V3: now also TP1.TP; no longer TP1.1
- net 5.2V: now also TP2.TP; no longer TP2.1
- net GND: now also TP3.TP; no longer TP3.1
Routing:
- net 5.2V: track 22.1 -> 40.4 mm
- net GND: track 32.8 -> 43.9 mm, vias 1 -> 3
- net 3V3: track 102.1 -> 105.7 mm
Changed lines of the file:
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@@
 <attribute name="VALUE" x="14.605" y="19.7612" size="1.27" layer="27" ratio="6" rot="SR270"/>
 </element>
-<element name="TP1" library="SparkFun-Connectors" library_urn="urn:adsk.eagle:library:513" package="1X01" package3d_urn="urn:adsk.eagle:package:38028/2" value="" x="1.905" y="17.907" smashed="yes">
-<attribute name="NAME" x="0.635" y="19.304" size="0.6096" layer="25" font="vector" ratio="20"/>
-<attribute name="VALUE" x="0.635" y="16.383" size="0.6096" layer="27" font="vector" ratio="20" align="top-left"/>
+<element name="TP1" library="X16-ExtraComponents" package="TESTPOINT_5.04MM" value="TESTPOINT_5.04MM" x="4.064" y="22.86" smashed="yes">
+<attribute name="NAME" x="1.524" y="25.781" size="1.27" layer="25" ratio="10"/>
+<attribute name="VALUE" x="2.794" y="21.463" size="0.0254" layer="27"/>
 </element>
-<element name="TP2" library="SparkFun-Connectors" library_urn="urn:adsk.eagle:library:513" package="1X01" package3d_urn="urn:adsk.eagle:package:38028/2" value="" x="11.049" y="2.667" smashed="yes">
-<attribute name="NAME" x="9.779" y="4.064" size="0.6096" layer="25" font="vector" ratio="20"/>
-<attribute name="VALUE" x="9.779" y="1.143" size="0.6096" layer="27" font="vector" ratio="20" align="top-left"/>
+<element name="TP2" library="X16-ExtraComponents" package="TESTPOINT_5.04MM" value="TESTPOINT_5.04MM" x="7.874" y="3.81" smashed="yes">
+<attribute name="NAME" x="5.334" y="6.731" size="1.27" layer="25" ratio="10"/>
+<attribute name="VALUE" x="6.604" y="2.413" size="0.0254" layer="27"/>
 </element>
-<element name="TP3" library="SparkFun-Connectors" library_urn="urn:adsk.eagle:library:513" package="1X01" package3d_urn="urn:adsk.eagle:package:38028/2" value="" x="2.159" y="31.115" smashed="yes">
-<attribute name="NAME" x="0.889" y="32.512" size="0.6096" layer="25" font="vector" ratio="20"/>
-<attribute name="VALUE" x="0.889" y="29.591" size="0.6096" layer="27" font="vector" ratio="20" align="top-left"/>
+<element name="TP3" library="X16-ExtraComponents" package="TESTPOINT_5.04MM" value="TESTPOINT_5.04MM" x="4.064" y="30.099" smashed="yes">
+<attribute name="NAME" x="1.524" y="33.02" size="1.27" layer="25" ratio="10"/>
+<attribute name="VALUE" x="2.794" y="28.702" size="0.0254" layer="27"/>
 </element>
 </elements>
@@
 <contactref element="U$2" pad="VSS1"/>
 <contactref element="D1" pad="C"/>
-<contactref element="TP3" pad="1"/>
 <polygon width="0.1524" layer="1">
 <vertex x="-1.651" y="36.322"/>
@@
 <wire x1="33.274" y1="19.089" x2="33.528" y2="19.343" width="0.2032" layer="16"/>
 <wire x1="33.528" y1="19.343" x2="31.242" y2="19.343" width="0.2032" layer="16"/>
-<wire x1="31.168" y1="22.544" x2="31.242" y2="22.544" width="0.2032" layer="1"/>
-<wire x1="31.242" y1="22.544" x2="31.968" y2="22.544" width="0.2032" layer="1"/>
+<wire x1="31.168" y1="22.544" x2="31.968" y2="22.544" width="0.2032" layer="1"/>
 <wire x1="48.895" y1="32.385" x2="46.355" y2="29.845" width="0.2032" layer="1"/>
 <wire x1="46.355" y1="24.003" x2="48.895" y2="21.463" width="0.2032" layer="1"/>
@@
 <wire x1="36.768" y1="14.706" x2="36.768" y2="14.044" width="0.2032" layer="1"/>
 <wire x1="36.576" y1="14.898" x2="36.768" y2="14.706" width="0.2032" layer="1"/>
+<contactref element="TP3" pad="TP"/>
+<wire x1="8.89" y1="19.773" x2="7.405" y2="19.773" width="0.2032" layer="1"/>
+<wire x1="7.405" y1="19.773" x2="7.366" y2="19.812" width="0.2032" layer="1"/>
+<via x="7.366" y="19.812" extent="1-16" drill="0.35"/>
+<wire x1="7.366" y1="19.812" x2="6.096" y2="18.542" width="0.2032" layer="16"/>
+<wire x1="6.096" y1="18.542" x2="6.096" y2="14.224" width="0.2032" layer="16"/>
+<wire x1="6.096" y1="14.224" x2="6.604" y2="13.716" width="0.2032" layer="16"/>
+<wire x1="6.604" y1="13.716" x2="7.874" y2="13.716" width="0.2032" layer="16"/>
+<via x="7.874" y="13.716" extent="1-16" drill="0.35"/>
+<wire x1="7.874" y1="13.716" x2="8.167" y2="14.009" width="0.2032" layer="1"/>
+<wire x1="8.167" y1="14.009" x2="9.144" y2="14.009" width="0.2032" layer="1"/>
 </signal>
 <signal name="TIM2_CH1">
@@
 <contactref element="J5" pad="2"/>
 <contactref element="J4" pad="5"/>
-<contactref element="TP1" pad="1"/>
 <wire x1="33.528" y1="21.043" x2="31.242" y2="21.043" width="0.508" layer="16"/>
 <wire x1="31.242" y1="21.043" x2="28.233" y2="21.043" width="0.508" layer="16"/>
@@
 <wire x1="8.89" y1="18.073" x2="11.9752" y2="18.073" width="0.508" layer="1"/>
 <wire x1="11.9752" y1="18.073" x2="12.0142" y2="18.034" width="0.508" layer="1"/>
-<wire x1="8.89" y1="18.073" x2="2.071" y2="18.073" width="0.508" layer="1"/>
-<wire x1="2.071" y1="18.073" x2="1.905" y2="17.907" width="0.508" layer="1"/>
-<wire x1="1.905" y1="17.907" x2="1.905" y2="10.021" width="0.508" layer="1"/>
-<wire x1="1.905" y1="10.021" x2="2.032" y2="9.894" width="0.508" layer="1"/>
+<wire x1="8.89" y1="18.073" x2="4.318" y2="18.073" width="0.508" layer="1"/>
+<wire x1="4.318" y1="18.073" x2="4.064" y2="18.073" width="0.508" layer="1"/>
 <wire x1="42.799" y1="12.954" x2="42.799" y2="14.605" width="0.508" layer="16"/>
 <wire x1="42.799" y1="14.605" x2="42.037" y2="15.367" width="0.508" layer="16"/>
@@
 <wire x1="38.218" y1="15.494" x2="39.243" y2="15.494" width="0.508" layer="1"/>
 <wire x1="39.243" y1="15.494" x2="39.37" y2="15.367" width="0.508" layer="1"/>
+<contactref element="TP1" pad="TP"/>
+<wire x1="4.318" y1="22.606" x2="4.064" y2="22.86" width="0.508" layer="1"/>
+<wire x1="4.318" y1="22.606" x2="4.318" y2="18.073" width="0.508" layer="1"/>
+<wire x1="2.032" y1="9.894" x2="2.032" y2="16.041" width="0.508" layer="1"/>
+<wire x1="2.032" y1="16.041" x2="4.064" y2="18.073" width="0.508" layer="1"/>
 </signal>
 <signal name="5.2V">
@@
 <contactref element="U1" pad="3"/>
 <contactref element="C5" pad="2"/>
-<contactref element="TP2" pad="1"/>
-<wire x1="14.732" y1="2.54" x2="11.176" y2="2.54" width="0.508" layer="1"/>
-<wire x1="11.176" y1="2.54" x2="11.049" y2="2.667" width="0.508" layer="1"/>
 <wire x1="14.732" y1="2.54" x2="16.732" y2="2.54" width="0.508" layer="1"/>
-<wire x1="9.169" y1="15.734" x2="12.0142" y2="15.734" width="0.508" layer="1"/>
-<wire x1="9.169" y1="15.734" x2="9.144" y2="15.709" width="0.508" layer="1"/>
-<wire x1="12.0142" y1="6.477" x2="12.0142" y2="15.734" width="0.508" layer="1"/>
-<wire x1="11.049" y1="2.667" x2="11.049" y2="5.5118" width="0.508" layer="1"/>
-<wire x1="11.049" y1="5.5118" x2="12.0142" y2="6.477" width="0.508" layer="1"/>
+<wire x1="12.0142" y1="15.734" x2="12.0142" y2="6.477" width="0.508" layer="1"/>
+<contactref element="TP2" pad="TP"/>
+<wire x1="9.144" y1="15.709" x2="8.089" y2="15.709" width="0.508" layer="1"/>
+<wire x1="9.144" y1="2.54" x2="14.732" y2="2.54" width="0.508" layer="1"/>
+<wire x1="11.9892" y1="15.709" x2="12.0142" y2="15.734" width="0.508" layer="1"/>
+<wire x1="9.144" y1="2.54" x2="8.5725" y2="3.1115" width="0.508" layer="1"/>
+<wire x1="8.5725" y1="3.1115" x2="7.874" y2="3.81" width="0.508" layer="1"/>
+<wire x1="6.858" y1="14.478" x2="6.858" y2="4.572" width="0.508" layer="1"/>
+<wire x1="6.858" y1="4.572" x2="7.62" y2="3.81" width="0.508" layer="1"/>
+<wire x1="7.62" y1="3.81" x2="7.874" y2="3.81" width="0.508" layer="1"/>
+<wire x1="8.089" y1="15.709" x2="6.858" y2="14.478" width="0.508" layer="1"/>
+<wire x1="12.0142" y1="6.477" x2="8.6487" y2="3.1115" width="0.508" layer="1"/>
+<wire x1="8.6487" y1="3.1115" x2="8.5725" y2="3.1115" width="0.508" layer="1"/>
+<wire x1="9.144" y1="15.709" x2="11.9892" y2="15.709" width="0.508" layer="1"/>
 </signal>
 <signal name="SWCLK">

Commit message: 12/16/2023
Parts:
- removed J4: (no value), SparkFun-Connectors:1X05_LOCK
- removed J5: (no value), SparkFun-Connectors:1X02
- added JP1: (no value), X16-ExtraComponents:1X05
- added JP2: (no value), X16-ExtraComponents:1X02
- moved J6 2.04 mm to (14.9, 4.57), flipped to the bottom, turned to 180 degrees
- moved R1 1.69 mm to (46.0, 11.8), turned to 90 degrees
- moved C5 1.17 mm to (10.3, 15.1)
- moved C7 1.17 mm to (10.0, 19.2)
- moved C3 1.08 mm to (46.0, 7.75)
- moved J2 0.25 mm to (36.6, 2.54)
- moved C2 0.13 mm to (33.3, 16.9)
- moved C6 0.13 mm to (35.3, 16.9)
Connections:
- net 3V3: now also JP1.5, JP2.2, R1.2; no longer J4.5, J5.2, R1.1
- net GND: now also JP1.3, JP2.1; no longer J4.3, J5.1
- net NRST: now also JP1.1, R1.1; no longer J4.1, R1.2
- net SWCLK: now also JP1.4; no longer J4.4
- net SWDIO: now also JP1.2; no longer J4.2
Routing:
- net GND: track 43.9 -> 86.2 mm, vias 3 -> 8
- net 5.2V: track 40.4 -> 25.0 mm
- net NRST: track 45.2 -> 56.4 mm, vias 0 -> 2
- net TIM1_CH3: track 26.2 -> 35.6 mm, vias 0 -> 2
- net TIM1_CH4: track 26.9 -> 34.2 mm, vias 1 -> 2
- net TIM3_CH1: track 49.5 -> 43.1 mm, vias 0 -> 3
- net MISO: track 32.7 -> 26.3 mm, vias 2 -> 1
- net SWCLK: track 18.3 -> 12.0 mm
- net 3V3: track 105.7 -> 99.4 mm, vias 5 -> 4
- net TIM2_CH1: track 38.1 -> 42.0 mm
- net SWDIO: track 16.1 -> 12.8 mm
- net TIM3_CH2: track 46.4 -> 49.6 mm, vias 0 -> 3
- net TIM2_CH2: track 37.5 -> 40.3 mm
- net TIM1_CH1: track 48.4 -> 45.7 mm, vias 2 -> 3
- net SCLK: track 21.8 -> 19.2 mm, vias 0 -> 1
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Other:
- board text added: "GND"
